File: kicad/gd-keypad-pcb/gd-keypad.kicad_pcb (KiCad board)
At the start: 2 copper layers, 58 parts, among them J2 USB_C_Receptacle_USB2.0_16P, J3 TC2030, SW1 TS-1187A-B-A-B, SW2 TS-1187A-B-A-B, SW3 RotaryEncoder_Switch_MP, U1 AT32F405RCT7, U2 USBLC6-2SC6, U3 TLV75733PDBV, U4 XC6206P332MR-G, U5 SW_MX_HE, U6 SW_MX_HE, U7 SW_MX_HE, Y1 X322512MSB4SI

Commit message: updated pcb
Parts:
- added G***: LOGO, logos:gd_ufo, F.Cu at (104.0, 124.7)
- added G***: LOGO, logos:gd_cube_cut+edited, F.Cu at (103.9, 123.7)
- moved C9 90.2 mm to (189.4, 67.8)
- moved C7 88.2 mm to (190.3, 87.4), turned to 0 degrees
- moved C5 88.0 mm to (186.5, 104.2), turned to 0 degrees
- moved C6 88.0 mm to (186.5, 109.7)
- moved C8 82.3 mm to (184.4, 87.4), turned to 0 degrees
- moved C4 52.7 mm to (148.5, 109.7)
- moved C3 51.6 mm to (148.5, 104.2), turned to 0 degrees
- moved C150 51.4 mm to (94.6, 73.5), turned to 90 degrees
- moved U4 50.3 mm to (97.3, 72.8), turned to -90 degrees
- moved C151 48.4 mm to (97.3, 69.5)
- moved C148 41.4 mm to (105.4, 73.0), turned to 90 degrees
- moved U3 38.6 mm to (109.0, 72.7), turned to 0 degrees
- moved R4 38.2 mm to (154.6, 76.6), turned to 90 degrees
- moved C149 34.3 mm to (112.2, 73.0), turned to 90 degrees
- moved R3 33.0 mm to (103.5, 95.9), turned to 90 degrees
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Connections:
- U1 pad 14: HE SENSOR 1 -> HE SENSOR 3
- U1 pad 16: HE SENSOR 3 -> HE SENSOR 1
- U1 pad 17: unconnected-(U1-PA3-Pad17) -> ENCODER S1
- U1 pad 18: unconnected-(U1-PF4-Pad18) -> ENCODER A
- U1 pad 19: unconnected-(U1-PF5-Pad19) -> ENCODER B
- U1 pad 21: COLUMN 0 -> COLUMN 1
- U1 pad 22: COLUMN 1 -> COLUMN 0
- U1 pad 24: ROW 0 -> ROW 2
- U1 pad 26: ROW 2 -> ROW 0
- U1 pad 28: ENCODER A -> unconnected-(U1-PB2-Pad28)
- U1 pad 29: ENCODER B -> unconnected-(U1-PB10-Pad29)
- U1 pad 30: ENCODER S1 -> unconnected-(U1-PB12-Pad30)
Routing:
- net SWDIO: track 0.00 -> 119.9 mm, vias 0 -> 2
- net SWCLK: track 0.00 -> 106.3 mm, vias 0 -> 2
- net ENCODER S1: track 0.00 -> 101.6 mm, vias 0 -> 2
- net SWO: track 0.00 -> 92.0 mm, vias 0 -> 2
- net NRST: track 6.00 -> 96.1 mm
- net COLUMN 0: track 38.1 -> 125.0 mm, vias 0 -> 2
- net ENCODER B: track 0.00 -> 85.2 mm, vias 0 -> 2
- net HE SENSOR 3: track 0.00 -> 83.5 mm, vias 0 -> 2
- net ENCODER A: track 0.00 -> 79.6 mm, vias 0 -> 2
- net COLUMN 1: track 42.8 -> 106.7 mm, vias 0 -> 6
- net ROW 2: track 19.8 -> 77.9 mm
- net HE SENSOR 2: track 0.00 -> 46.9 mm, vias 0 -> 2
- net GND: track 3.18 -> 45.6 mm, vias 0 -> 34
- net USB_D-: track 0.00 -> 41.3 mm
- net BOOT0: track 6.00 -> 47.3 mm
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- added copper zone on B.Cu, net +3.3V
- added copper zone on B.Cu, net +5V
- added copper zone on B.Cu, net GND
- added copper zone on F.Cu, net GND
Other:
- board outline added: 152.5 x 68 mm
- board text added: "LouisDevice 3H6MGD"

Commit message: updated pcb design
Parts:
- added G***: LOGO, logos:gd_cube, F.Cu at (77.9, 94.0)
- moved C7 0.08 mm to (190.2, 87.4), turned to 180 degrees
- turned C8 to 180 degrees
Routing:
- net +3.3VA: track 12.1 -> 155.3 mm, vias 0 -> 2
- net HE SENSOR 3: track 83.5 -> 104.9 mm
- net GND: track 45.6 -> 55.1 mm, vias 34 -> 39
- net +5V: track 6.00 -> 11.2 mm
- net HE SENSOR 2: track 46.9 -> 49.9 mm
- net ENCODER B: track 85.2 -> 87.1 mm
- net +3.3V: track 22.9 -> 24.3 mm
- net NRST: track 96.1 -> 95.5 mm, vias 0 -> 2
- net SWO: track 92.0 -> 92.2 mm, vias 2 -> 4
- net SWDIO: track 119.9 -> 119.8 mm, vias 2 -> 4
- net SWCLK: vias 2 -> 4
- added copper zone on B.Cu, net +3.3VA
Other:
- board text added: "3H6MGD"

Commit message: updated pcb design
Parts:
- moved J3 80.9 mm to (168.0, 71.0), turned to 0 degrees
- moved C6 70.3 mm to (117.7, 95.5), turned to 90 degrees
- moved C4 35.2 mm to (116.1, 95.9), turned to 90 degrees
- moved C2 13.6 mm to (114.4, 96.7), turned to 90 degrees
- moved R4 4.13 mm to (154.8, 72.5)
- moved SW1 4.13 mm to (150.2, 78.5)
- moved SW2 4.13 mm to (150.2, 71.1)
- moved C152 0.69 mm to (117.8, 87.1)
- moved C153 0.69 mm to (124.7, 87.1)
- moved Y1 0.69 mm to (121.3, 87.4)
- moved H3 0.25 mm to (195.4, 66.4)
Routing:
- net SWDIO: track 119.8 -> 76.6 mm, vias 4 -> 2
- net SWCLK: track 106.3 -> 70.7 mm, vias 4 -> 2
- net SWO: track 92.2 -> 71.3 mm, vias 4 -> 2
- net NRST: track 95.5 -> 87.7 mm, vias 2 -> 0
- net +3.3VA: track 155.3 -> 162.1 mm, vias 2 -> 4
- net HE SENSOR 3: track 104.9 -> 98.3 mm
- net HE SENSOR 1: track 25.1 -> 21.2 mm
- net +3.3V: track 24.3 -> 28.1 mm
- net BOOT0: track 47.3 -> 50.1 mm
- net ENCODER S1: track 101.6 -> 104.3 mm
- net ENCODER B: track 87.1 -> 89.3 mm
- net ENCODER A: track 79.4 -> 81.5 mm
- net GND: track 55.1 -> 53.4 mm, vias 39 -> 40
- net HE SENSOR 2: track 49.9 -> 49.0 mm

Commit message: updated pcb design
Parts:
- moved H3 177.9 mm to (18.0, 79.2)
- moved H2 159.4 mm to (164.9, 18.0)
- moved H5 120.8 mm to (96.2, 58.3)
- moved C7 117.5 mm to (78.6, 50.6)
- moved C8 110.0 mm to (81.0, 50.0), turned to 90 degrees
- moved C9 108.3 mm to (82.6, 49.9), turned to 0 degrees
- moved C160 61.6 mm to (86.9, 41.8), turned to 90 degrees
- moved SW3 59.6 mm to (153.3, 28.5)
- moved J2 59.6 mm to (91.0, 17.6)
- moved R4 58.3 mm to (123.1, 23.6)
- moved C1 58.3 mm to (78.6, 55.2)
- moved C148 58.3 mm to (73.8, 24.1)
- moved C149 58.3 mm to (80.5, 24.1)
- moved C150 58.3 mm to (62.9, 24.6)
- moved C3 58.3 mm to (116.8, 55.2)
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Routing:
- net +3.3V: track 28.1 -> 43.9 mm, vias 2 -> 4
- net ENCODER S1: track 104.3 -> 100.9 mm
- net USB_PLUG_D+: track 6.65 -> 9.10 mm
- net VBUS: track 10.3 -> 12.0 mm
- net Net-(J2-CC2): track 2.41 -> 4.03 mm
- net Net-(J2-CC1): track 2.61 -> 4.23 mm
- net USB_PLUG_D-: track 7.88 -> 9.42 mm
- net ENCODER A: track 81.5 -> 83.0 mm
- net ENCODER B: track 89.3 -> 90.7 mm
- net GND: track 53.4 -> 54.5 mm, vias 40 -> 42
- net NRST: track 87.7 -> 88.6 mm
- net HE SENSOR 2: track 49.0 -> 48.4 mm
- net SWO: track 71.3 -> 70.8 mm
Other:
- board size 152.5 x 68 mm -> 155.1 x 69.2 mm

Commit message: finalized pcb design
Parts:
- MX1, MX2, MX3, MX4, MX5, MX6: footprint PCM_marbastlib-mx:SW_MX_HS_CPG151101S11_1u -> PCM_marbastlib-mx:SW_MX_HS_KS-2P02B01-01_1u
- moved H1 0.43 mm to (17.9, 17.6)
- moved H3 0.43 mm to (17.9, 79.6)
- moved H4 0.43 mm to (164.9, 79.6)
- moved H2 0.43 mm to (164.9, 17.6)
- moved H5 0.17 mm to (96.2, 58.1)
- moved H6 0.13 mm to (134.3, 58.1)
Routing:
- net Net-(D5-A): track 12.6 -> 14.8 mm
- net Net-(D1-A): track 12.6 -> 14.8 mm
- net Net-(D3-A): track 12.6 -> 14.8 mm
- net Net-(D4-A): track 12.6 -> 14.8 mm
- net Net-(D6-A): track 12.6 -> 14.8 mm
- net Net-(D2-A): track 12.6 -> 14.8 mm
- net ROW 1: track 58.8 -> 60.4 mm
- net ROW 2: track 78.1 -> 79.5 mm
- net ROW 0: track 60.1 -> 61.1 mm
- net SWO: track 70.8 -> 70.2 mm
Other:
- board size 155.1 x 69.2 mm -> 155 x 70 mm
