File: kicad/gd-keypad-pcb/gd-keypad.kicad_sch (KiCad schematic)
At the start: 58 parts, among them J1 TYPE-C-31-M-12, J3 TC2030, SW1 TS-1187A-B-A-B, SW2 TS-1187A-B-A-B, SW3 RotaryEncoder_Switch_MP, U1 AT32F405RCT7, U2 USBLC6-2SC6, U3 TLV75733PDBV, U4 XC6206P332MR-G, U5 SW_MX_HE, U6 SW_MX_HE, U7 SW_MX_HE, Y1 X322512MSB4SI

Commit message: schematic completed
Parts:
- removed J1: TYPE-C-31-M-12, Connector_USB:USB_C_Receptacle_HRO_TYPE-C-31-M-12, symbol Connector:USB_C_Receptacle_USB2.0_16P
- added J2: USB_C_Receptacle_USB2.0_16P, Connector_USB:USB_C_Receptacle_HRO_TYPE-C-31-M-12, symbol Connector:USB_C_Receptacle_USB2.0_16P
- C1, C2, C3, C4, C5, C6, C7, C8, C9: footprint (none) -> Capacitor_SMD:C_0402_1005Metric
- H1, H2, H3, H4, H5, H6: footprint (none) -> MountingHole:MountingHole_2.7mm_M2.5_DIN965_Pad
- SW3: footprint (none) -> PCM_marbastlib-various:ROT_Alps_EC11E-Switch
- Y1: private (none) -> KLC_S4.1
Connections:
- net GNDA is gone; now on net GND: C1.2, C3.2, C5.2
- net GND: now also J2.A1 (GND), J2.A12 (GND), J2.B1 (GND), J2.B12 (GND), J2.SH (SHIELD)
- net USB_PLUG_D+: now also J2.A6 (D+), J2.B6 (D+)
- net USB_PLUG_D-: now also J2.A7 (D-), J2.B7 (D-)
- net VBUS: now also J2.A4 (VBUS), J2.A9 (VBUS), J2.B4 (VBUS), J2.B9 (VBUS)
- net at R1.1: now also J2.A5 (CC1)
- net at R2.2: now also J2.B5 (CC2)
Other:
- moved on the sheet: C1, C2, C3, C4, C5, C6, C7, C8, C9, D1, D2, D3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

Commit message: completed pcb schematic
Parts:
- removed MX1, MX2, MX3, MX4, MX5, MX6: MX_SW_solder, PCM_marbastlib-mx:SW_MX_1u, symbol PCM_marbastlib-mx:MX_SW_solder
- added MX1, MX2, MX3, MX4, MX5, MX6: MX_SW_HS, PCM_marbastlib-mx:SW_MX_HS_CPG151101S11_1u, symbol PCM_marbastlib-mx:MX_SW_HS_CPG151101S11
Connections:
- net COLUMN 0: now also MX1.1, MX3.1, MX5.1
- net COLUMN 1: now also MX2.1, MX4.1, MX6.1
- net at D3.2 (A): now also MX3.2
- net at D2.2 (A): now also MX2.2
- net at D6.2 (A): now also MX6.2
- net at D4.2 (A): now also MX4.2
- net at D5.2 (A): now also MX5.2
- net at D1.2 (A): now also MX1.2

Commit message: updated pcb
Connections:
- net COLUMN 0: now also U1.22 (PA6); no longer U1.21 (PA5)
- net COLUMN 1: now also U1.21 (PA5); no longer U1.22 (PA6)
- net ENCODER A: now also U1.18 (PF4); no longer U1.28 (PB2)
- net ENCODER B: now also U1.19 (PF5); no longer U1.29 (PB10)
- net ENCODER S1: now also U1.17 (PA3); no longer U1.30 (PB12)
- net HE SENSOR 1: now also U1.16 (PA2); no longer U1.14 (PA0)
- net HE SENSOR 3: now also U1.14 (PA0); no longer U1.16 (PA2)
- net ROW 0: now also U1.26 (PB0); no longer U1.24 (PC4)
- net ROW 2: now also U1.24 (PC4); no longer U1.26 (PB0)

Commit message: finalized pcb design
Parts:
- removed MX1, MX2, MX3, MX4, MX5, MX6: MX_SW_HS, PCM_marbastlib-mx:SW_MX_HS_CPG151101S11_1u, symbol PCM_marbastlib-mx:MX_SW_HS_CPG151101S11
- added MX1, MX2, MX3, MX4, MX5, MX6: MX_SW_HS, PCM_marbastlib-mx:SW_MX_HS_KS-2P02B01-01_1u, symbol PCM_marbastlib-mx:MX_SW_HS_KS-2P02B01-01
Connections:
- net COLUMN 0: now also MX1.1, MX3.1, MX5.1
- net COLUMN 1: now also MX2.1, MX4.1, MX6.1
- net at D3.2 (A): now also MX3.2
- net at D4.2 (A): now also MX4.2
- net at D2.2 (A): now also MX2.2
- net at D6.2 (A): now also MX6.2
- net at D5.2 (A): now also MX5.2
- net at D1.2 (A): now also MX1.2
